Commit message: fix laser link orientation

File: Mobile Robot Demo/Assets/URDF/fetch_description/urdf/freight.urdf.xacro (robot description, xacro)
@@ -135,5 +135,5 @@
     </link>
     <joint name="${prefix}laser_joint" type="fixed">
-      <origin rpy="3.14159265359 0 0" xyz="0.235 0 0.2878" />
+      <origin rpy="0 0 0" xyz="0.235 0 0.2878" />
       <parent link="${prefix}chassis_link" />
       <child link="${prefix}laser_link" />

File: Mobile Robot Demo/Assets/URDF/freight.urdf (robot description, URDF)
Before this commit: robot Freight, 8 links, 7 joints
Joints:
- joint freight/laser_joint: origin xyz=0.235 0 0.2878 rpy=3.14159265359 0 0 -> xyz=0.235 0 0.2878 rpy=0 0 0

Commit message: update to latest version

File: Mobile Robot Demo/Assets/URDF/fetch_description/urdf/freight.urdf.xacro (robot description, xacro)
@@ -135,5 +135,5 @@
     </link>
     <joint name="${prefix}laser_joint" type="fixed">
-      <origin rpy="0 0 0" xyz="0.235 0 0.2878" />
+      <origin rpy="3.14159265359 0 0" xyz="0.235 0 0.2878" />
       <parent link="${prefix}chassis_link" />
       <child link="${prefix}laser_link" />

File: Mobile Robot Demo/Assets/URDF/freight.urdf (robot description, URDF)
Before this commit: robot Freight, 8 links, 7 joints
Joints:
- joint freight/laser_joint: origin xyz=0.235 0 0.2878 rpy=0 0 0 -> xyz=0.235 0 0.2878 rpy=3.14159265359 0 0

Commit message: update to latest version

File: Mobile Robot Demo/Assets/URDF/fetch_description/urdf/freight.urdf.xacro (robot description, xacro)
@@ -135,5 +135,5 @@
     </link>
     <joint name="${prefix}laser_joint" type="fixed">
-      <origin rpy="0 0 0" xyz="0.235 0 0.2878" />
+      <origin rpy="3.141592653589793 0 0" xyz="0.235 0 0.2878" />
       <parent link="${prefix}chassis_link" />
       <child link="${prefix}laser_link" />

File: Mobile Robot Demo/Assets/URDF/freight.urdf (robot description, URDF)
Before this commit: robot Freight, 8 links, 7 joints
Joints:
- joint freight/laser_joint: origin xyz=0.235 0 0.2878 rpy=0 0 0 -> xyz=0.235 0 0.2878 rpy=3.141592653589793 0 0
